File: hardware/rev3/LOLRGB_3.brd (EAGLE design)
At the start: 31.9 x 17.8 mm, 77 parts, among them Q1 BSS138

Commit message: SOT23-Footprint changed
Parts:
- Q1: device transistor-small-signal:SOT23 -> adafruit:SOT23-R
- moved Q1 0.11 mm to (12.3, 7.00)
Changed lines of the file:
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@@
 <attribute name="VALUE" x="10.395" y="-6.465" size="0.8128" layer="27" rot="R270"/>
-</element>
-<element name="Q1" library="transistor-small-signal" package="SOT23" value="BSS138" x="12.3952" y="7.0508" smashed="yes" rot="R270">
-<attribute name="VALUE" x="9.2202" y="8.9558" size="1.27" layer="27" rot="R270"/>
 </element>
 <element name="R1" library="rcl" package="ADAFRUIT_R0402-VISHAY" value="10k" x="10.0124" y="7.5434" rot="R90"/>
 <element name="R2" library="rcl" package="ADAFRUIT_R0402-VISHAY" value="10k" x="14.764" y="6.6048" rot="R270"/>
+<element name="Q1" library="adafruit" package="SOT23-R" value="BSS138" x="12.3" y="7" rot="R270"/>
 </elements>
 <signals>
@@
 <contactref element="LEFT" pad="6"/>
 <contactref element="R1" pad="1"/>
-<contactref element="Q1" pad="2"/>
 <wire x1="10.0124" y1="7.0934" x2="10.837946875" y2="7.0934" width="0.2" layer="1"/>
 <wire x1="10.837946875" y1="7.0934" x2="11.14326875" y2="6.96693125" width="0.2" layer="1" curve="-45"/>
 <wire x1="11.14326875" y1="6.96693125" x2="11.208628125" y2="6.901571875" width="0.2" layer="1"/>
 <wire x1="11.208628125" y1="6.901571875" x2="11.2952" y2="6.69256875" width="0.2" layer="1" curve="-44.999394"/>
-<wire x1="11.2952" y1="6.69256875" x2="11.2952" y2="6.1008" width="0.2" layer="1"/>
 <wire x1="10.0124" y1="7.0934" x2="9.667496875" y2="7.0934" width="0.2" layer="1"/>
 <wire x1="9.667496875" y1="7.0934" x2="9.349125" y2="6.961525" width="0.2" layer="1" curve="45"/>
@@
 <wire x1="0.27459375" y1="6.477" x2="-1.38658125" y2="7.16508125" width="0.2" layer="1" curve="-44.999946"/>
 <wire x1="-1.38658125" y1="7.16508125" x2="-1.8542" y2="7.6327" width="0.2" layer="1"/>
+<contactref element="Q1" pad="2"/>
+<wire x1="11.2952" y1="6.69256875" x2="11.3" y2="6.69256875" width="0.2" layer="1"/>
+<wire x1="11.3" y1="6.69256875" x2="11.3" y2="6.05" width="0.2" layer="1"/>
 </signal>
 <signal name="GPIO15">
@@
 <contactref element="LEFT" pad="4"/>
 <contactref element="R1" pad="2"/>
-<contactref element="Q1" pad="1"/>
 <via x="12.4714" y="8.2296" extent="1-16" drill="0.254"/>
 <wire x1="12.4714" y1="8.2296" x2="11.52918125" y2="8.2296" width="0.2" layer="16"/>
@@
 <wire x1="-4.518515625" y1="6.477" x2="-6.66944375" y2="7.36794375" width="0.2" layer="16" curve="-45"/>
 <wire x1="-6.66944375" y1="7.36794375" x2="-6.9342" y2="7.6327" width="0.2" layer="16"/>
-<wire x1="11.2952" y1="8.0008" x2="11.524" y2="8.2296" width="0.2" layer="1"/>
-<wire x1="11.524" y1="8.2296" x2="12.4714" y2="8.2296" width="0.2" layer="1"/>
 <wire x1="10.0124" y1="7.9934" x2="10.0124" y2="8.0008" width="0.2" layer="1"/>
-<wire x1="10.0124" y1="8.0008" x2="11.2952" y2="8.0008" width="0.2" layer="1"/>
+<contactref element="Q1" pad="1"/>
+<wire x1="10.0124" y1="7.9934" x2="11.2434" y2="7.9934" width="0.2" layer="1"/>
+<wire x1="11.2434" y1="7.9934" x2="11.3" y2="7.95" width="0.2" layer="1"/>
+<wire x1="11.3" y1="7.95" x2="11.796384375" y2="7.95" width="0.2" layer="1"/>
+<wire x1="11.796384375" y1="7.95" x2="12.4714" y2="8.2296" width="0.2" layer="1" curve="45"/>
 </signal>
 <signal name="LED_IN">
 <contactref element="LED1" pad="DIN"/>
 <contactref element="R2" pad="1"/>
-<contactref element="Q1" pad="3"/>
-<wire x1="13.7596" y1="7.3152" x2="13.4952" y2="7.0508" width="0.2" layer="1"/>
-<wire x1="13.4952" y1="7.0508" x2="13.4952" y2="7.3952" width="0.2" layer="1"/>
 <via x="14.7" y="7.75" extent="1-16" drill="0.254"/>
 <wire x1="14.764" y1="7.0548" x2="14.76" y2="7.0508" width="0.2" layer="1"/>
-<wire x1="14.76" y1="7.0508" x2="13.4952" y2="7.0508" width="0.2" layer="1"/>
 <wire x1="14.764" y1="7.0548" x2="14.7" y2="7.1188" width="0.2" layer="1"/>
 <wire x1="14.7" y1="7.1188" x2="14.7" y2="7.75" width="0.2" layer="1"/>
@@
 <via x="-8.4" y="6" extent="1-16" drill="0.254"/>
 <wire x1="-8.4" y1="6" x2="-8.641421875" y2="5.9" width="0.2" layer="1" curve="-45"/>
+<contactref element="Q1" pad="3"/>
+<wire x1="13.3" y1="7" x2="13.3452" y2="7.0548" width="0.2" layer="1"/>
+<wire x1="13.3452" y1="7.0548" x2="14.764" y2="7.0548" width="0.2" layer="1"/>
 </signal>
 </signals>
